Commit message: Changed laser link name

File: create_description/urdf/rplidar.urdf.xacro (robot description, xacro)
@@ -1,5 +1,5 @@
 <robot name="sensor_rplidar" xmlns:xacro="http://ros.org/wiki/xacro">
 	<!-- Joints and Links, standard URDF stuff -->
-	<link name="rplidar_link">
+	<link name="laser">
 		<collision>
 			<origin xyz="0 0 0" rpy="0 0 0"/>
@@ -25,7 +25,7 @@
 		<origin xyz="0 0 0.1" rpy="0 0 0 "/>
 		<parent link="base_link"/>
-		<child link="rplidar_link"/>
+		<child link="laser"/>
 	</joint>
-<gazebo reference="rplidar_link">
+<gazebo reference="laser">
 	<sensor type="ray" name="head_rplidar_sensor">
 		<pose>0 0 0 0 0 0</pose>
@@ -54,5 +54,5 @@
 			<topic_name>/scan</topic_name>
             <output_type>sensor_msgs/LaserScan</output_type>
-			<frame_name>rplidar_link</frame_name>
+			<frame_name>laser</frame_name>
             <ros>
                 <namespace></namespace>
