Commit message: fixed camera frames

File: create_description/urdf/camera.urdf.xacro (robot description, xacro)
@@ -1,4 +1,4 @@
 <?xml version="1.0"?>
-<robot name="sensor_rplidar" xmlns:xacro="http://ros.org/wiki/xacro">
+<robot name="sensor_camera" xmlns:xacro="http://ros.org/wiki/xacro">
 	<!-- Joints and Links, standard URDF stuff -->
 	<link name="camera">
@@ -9,11 +9,4 @@
 			</geometry>
 		</collision>
-		<vision>
-			<origin xyz="0 0 0.1" rpy="1.5707 0 0" />
-			<geometry>
-				<box size="0.1 0.1 0.1" />
-				<meshfile name="package://create_description/meshes/rplidar.dae" scale="0.001 0.001 0.001" />
-			</geometry>
-		</vision>
 		<inertial>
 			<mass value="1e-5" />
@@ -24,8 +17,17 @@
 	<joint name="camera_joint" type="fixed">
 		<axis xyz="0 1 0" />
-		<origin xyz="0 0 0.1" rpy="0 0 0 " />
+		<origin xyz="0 0 0.15" rpy="0 0 0 " />
 		<parent link="base_link" />
 		<child link="camera" />
 	</joint>
+	<joint name="camera_optical_joint" type="fixed">
+		<!-- these values have to be these values otherwise the gazebo camera
+        image won't be aligned properly with the frame it is supposedly
+        originating from -->
+		<origin xyz="0 0 0" rpy="${-pi/2} 0 ${-pi/2}" />
+		<parent link="camera" />
+		<child link="camera_optical" />
+	</joint>
+	<link name="camera_optical"></link>
 	<gazebo reference="camera">
 		<sensor type="camera" name="george_cam">
@@ -38,8 +40,6 @@
 				<alwaysOn>true</alwaysOn>
 				<updateRate>0.0</updateRate>
-				<cameraName>george_cam</cameraName>
-				<imageTopicName>image_raw</imageTopicName>
-				<cameraInfoTopicName>camera_info</cameraInfoTopicName>
-				<frameName>camera</frameName>
+				<camera_name>george_cam</camera_name>
+				<frame_name>camera_optical</frame_name>
 				<hackBaseline>0.07</hackBaseline>
 				<distortionK1>0.0</distortionK1>

File: create_description/urdf/rplidar.urdf.xacro (robot description, xacro)
@@ -1,2 +1,3 @@
+<?xml version="1.0"?>
 <robot name="sensor_rplidar" xmlns:xacro="http://ros.org/wiki/xacro">
 	<!-- Joints and Links, standard URDF stuff -->
