Commit message: modified sim to work for ign

File: create_description/urdf/create_base.urdf.xacro (robot description, xacro)
@@ -27,7 +27,9 @@
       <child link="${prefix}_wheel_link" />
       <axis xyz="0 1 0" />
+      <dynamics damping="0.2" />
     </joint>
   </xacro:macro>
-  <xacro:macro name="create_base" params="diffdrive_update_rate:=40 wheel_separation wheel_radius:=0.036 wheel_width:=0.024 wheel_torque:=1.0 wheel_accel:=1.8 mass_kg:=3.5 base_diameter *mesh">
+  <xacro:macro name="create_base"
+    params="diffdrive_update_rate:=40 wheel_separation wheel_radius:=0.036 wheel_width:=0.024 wheel_torque:=1.0 wheel_accel:=1.8 mass_kg:=3.5 base_diameter *mesh">
     <xacro:include filename="$(find create_description)/urdf/create_base_gazebo.urdf.xacro" />
     <link name="base_footprint">
@@ -50,5 +52,5 @@
         <mass value="2" />
         <origin xyz="0 0 0.0" />
-        <inertia ixx="0.01" ixy="0.0" ixz="0.0" iyy="0.01" iyz="0.0" izz="0.5" />
+        <inertia ixx="0.5" ixy="0.0" ixz="0.0" iyy="0.5" iyz="0.0" izz="0.5" />
       </inertial>
       <visual>
@@ -90,5 +92,5 @@
         <mass value="0.01" />
         <origin xyz="0 0 0" />
-        <inertia ixx="1.0" ixy="0.0" ixz="0.0" iyy="0.01" iyz="0.0" izz="0.01" />
+        <inertia ixx="0.01" ixy="0.0" ixz="0.0" iyy="0.01" iyz="0.0" izz="0.01" />
       </inertial>
     </link>
@@ -130,7 +132,10 @@
       <child link="rightfront_cliff_sensor_link" />
     </joint>
-    <xacro:create_wheel prefix="left" y_offset="${wheel_separation / 2}" wheel_radius="${wheel_radius}" wheel_width="${wheel_width}" />
-    <xacro:create_wheel prefix="right" y_offset="${wheel_separation / -2}" wheel_radius="${wheel_radius}" wheel_width="${wheel_width}" />
-    <!--<link name="rear_wheel_link">
+    <xacro:create_wheel prefix="left" y_offset="${wheel_separation / 2}"
+      wheel_radius="${wheel_radius}" wheel_width="${wheel_width}" />
+    <xacro:create_wheel prefix="right" y_offset="${wheel_separation / -2}"
+      wheel_radius="${wheel_radius}" wheel_width="${wheel_width}" />
+    <!--<link
+    name="rear_wheel_link">
     <inertial>
       <origin xyz="0 0 0"/>

File: create_description/urdf/create_base_gazebo.urdf.xacro (robot description, xacro)
@@ -1,23 +1,33 @@
-<?xml version="1.0" ?>
+<?xml version="1.0"?>
 <robot xmlns:xacro="http://ros.org/wiki/xacro">
   <xacro:macro name="sim_create_base">
+    <ros2_control name="IgnitionSystem" type="system">
+      <hardware>
+        <plugin>ign_ros2_control/IgnitionSystem</plugin>
+      </hardware>
+      <joint name="left_wheel_joint">
+        <command_interface name="velocity">
+          <param name="min">-10</param>
+          <param name="max">10</param>
+        </command_interface>
+        <state_interface name="position" />
+        <state_interface name="velocity" />
+      </joint>
+      <joint name="right_wheel_joint">
+        <command_interface name="velocity">
+          <param name="min">-10</param>
+          <param name="max">10</param>
+        </command_interface>
+        <state_interface name="position" />
+        <state_interface name="velocity" />
+      </joint>
+    </ros2_control>
     <gazebo>
-      <plugin name="differential_drive_controller" filename="libgazebo_ros_diff_drive.so">
-        <always_on>true</always_on>
-        <update_rate>${diffdrive_update_rate}</update_rate>
-        <left_joint>left_wheel_joint</left_joint>
-        <right_joint>right_wheel_joint</right_joint>
-        <wheel_separation>${wheel_separation}</wheel_separation>
-        <wheel_diameter>${wheel_radius * 2}</wheel_diameter>
-        <wheel_torque>${wheel_torque}</wheel_torque>
-        <!--wheelAcceleration>${wheel_accel}</wheelAcceleration-->
-        <odometry_topic>odom</odometry_topic>
-        <odometry_frame>odom</odometry_frame>
-        <robot_base_frame>base_footprint</robot_base_frame>
-        <publish_wheel_tf>true</publish_wheel_tf>
-        <publish_odom_tf>true</publish_odom_tf>
-        <publish_odom>true</publish_odom>
-        <odometry_source>1</odometry_source> <!-- 0 for encoders -->
+      <!-- Joint state publisher -->
+      <plugin filename="ign_ros2_control-system" name="ign_ros2_control::IgnitionROS2ControlPlugin">
+        <parameters>$(find create_description)/config/diff_drive_controller_velocity.yaml</parameters>
       </plugin>
+    </gazebo>
+    <gazebo>
       <plugin name="p3d_base_controller" filename="libgazebo_ros_p3d.so">
         <always_on>true</always_on>
@@ -29,5 +39,6 @@
         <xyz_offsets>0 0 0</xyz_offsets>
         <rpy_offsets>0 0 0</rpy_offsets>
-        <!--<interface:position name="p3d_base_position"/>-->
+        <!--<interface:position
+        name="p3d_base_position"/>-->
       </plugin>
     </gazebo>
@@ -66,17 +77,17 @@
   </xacro:macro>
   <xacro:macro name="sim_imu">
-      <gazebo>
-          <sensor>
-      <plugin name="imu_controller" filename="libgazebo_ros_imu_sensor.so">
-        <always_on>true</always_on>
-        <update_rate>30</update_rate>
-        <body_name>gyro_link</body_name>
-        <topic_name>imu/data</topic_name>
-        <service_name>imu/is_calibrated</service_name>
-        <gaussian_noise>${0.0017*0.0017}</gaussian_noise>
-        <xyz_offsets>0 0 0</xyz_offsets>
-        <rpy_offsets>0 0 0</rpy_offsets>
-    </plugin>
-</sensor>
+    <gazebo>
+      <sensor>
+        <plugin name="imu_controller" filename="libgazebo_ros_imu_sensor.so">
+          <always_on>true</always_on>
+          <update_rate>30</update_rate>
+          <body_name>gyro_link</body_name>
+          <topic_name>imu/data</topic_name>
+          <service_name>imu/is_calibrated</service_name>
+          <gaussian_noise>${0.0017*0.0017}</gaussian_noise>
+          <xyz_offsets>0 0 0</xyz_offsets>
+          <rpy_offsets>0 0 0</rpy_offsets>
+        </plugin>
+      </sensor>
     </gazebo>
   </xacro:macro>

Commit message: actually supports ign now

File: create_description/urdf/create_base.urdf.xacro (robot description, xacro)
@@ -204,7 +204,7 @@
     <!-- Simulation sensors -->
     <xacro:sim_create_base />
-    <xacro:sim_create_wall_sensor />
-    <xacro:sim_create_cliff_sensors />
-    <xacro:sim_imu />
+    <!-- <xacro:sim_create_wall_sensor /> -->
+    <!-- <xacro:sim_create_cliff_sensors /> -->
+    <!-- <xacro:sim_imu /> -->
   </xacro:macro>
 </robot>

File: create_description/urdf/create_base_gazebo.urdf.xacro (robot description, xacro)
@@ -76,138 +76,3 @@
     </gazebo>
   </xacro:macro>
-  <xacro:macro name="sim_imu">
-    <gazebo>
-      <sensor>
-        <plugin name="imu_controller" filename="libgazebo_ros_imu_sensor.so">
-          <always_on>true</always_on>
-          <update_rate>30</update_rate>
-          <body_name>gyro_link</body_name>
-          <topic_name>imu/data</topic_name>
-          <service_name>imu/is_calibrated</service_name>
-          <gaussian_noise>${0.0017*0.0017}</gaussian_noise>
-          <xyz_offsets>0 0 0</xyz_offsets>
-          <rpy_offsets>0 0 0</rpy_offsets>
-        </plugin>
-      </sensor>
-    </gazebo>
-  </xacro:macro>
-  <xacro:macro name="sim_create_wall_sensor">
-    <gazebo reference="wall_sensor_link">
-      <sensor type="ray" name="wall_sensor">
-        <always_on>true</always_on>
-        <update_rate>20.0</update_rate>
-        <pose>0 0 0 0 0 0</pose>
-        <visualize>false</visualize>
-        <ray>
-          <scan>
-            <horizontal>
-              <samples>1</samples>
-              <resolution>1</resolution>
-              <min_angle>0</min_angle>
-              <max_angle>0</max_angle>
-            </horizontal>
-          </scan>
-          <range>
-            <min>0.0160</min>
-            <max>0.04</max>
-            <resolution>0.1</resolution>
-          </range>
-        </ray>
-      </sensor>
-    </gazebo>
-  </xacro:macro>
-  <xacro:macro name="sim_create_cliff_sensors">
-    <gazebo reference="left_cliff_sensor_link">
-      <sensor type="ray" name="left_cliff_sensor">
-        <always_on>true</always_on>
-        <update_rate>20.0</update_rate>
-        <pose>0 0 0 0 0 0</pose>
-        <visualize>false</visualize>
-        <ray>
-          <scan>
-            <horizontal>
-              <samples>1</samples>
-              <resolution>1</resolution>
-              <min_angle>0</min_angle>
-              <max_angle>0</max_angle>
-            </horizontal>
-          </scan>
-          <range>
-            <min>0.01</min>
-            <max>0.04</max>
-            <resolution>0.1</resolution>
-          </range>
-        </ray>
-      </sensor>
-    </gazebo>
-    <gazebo reference="right_cliff_sensor_link">
-      <sensor type="ray" name="right_cliff_sensor">
-        <always_on>true</always_on>
-        <update_rate>20.0</update_rate>
-        <pose>0 0 0 0 0 0</pose>
-        <visualize>false</visualize>
-        <ray>
-          <scan>
-            <horizontal>
-              <samples>1</samples>
-              <resolution>1</resolution>
-              <min_angle>0</min_angle>
-              <max_angle>0</max_angle>
-            </horizontal>
-          </scan>
-          <range>
-            <min>0.01</min>
-            <max>0.04</max>
-            <resolution>0.1</resolution>
-          </range>
-        </ray>
-      </sensor>
-    </gazebo>
-    <gazebo reference="leftfront_cliff_sensor_link">
-      <sensor type="ray" name="leftfront_cliff_sensor">
-        <always_on>true</always_on>
-        <update_rate>20.0</update_rate>
-        <pose>0 0 0 0 0 0</pose>
-        <visualize>false</visualize>
-        <ray>
-          <scan>
-            <horizontal>
-              <samples>1</samples>
-              <resolution>1</resolution>
-              <min_angle>0</min_angle>
-              <max_angle>0</max_angle>
-            </horizontal>
-          </scan>
-          <range>
-            <min>0.01</min>
-            <max>0.04</max>
-            <resolution>0.1</resolution>
-          </range>
-        </ray>
-      </sensor>
-    </gazebo>
-    <gazebo reference="rightfront_cliff_sensor_link">
-      <sensor type="ray" name="rightfront_cliff_sensor">
-        <always_on>true</always_on>
-        <update_rate>20.0</update_rate>
-        <pose>0 0 0 0 0 0</pose>
-        <visualize>false</visualize>
-        <ray>
-          <scan>
-            <horizontal>
-              <samples>1</samples>
-              <resolution>1</resolution>
-              <min_angle>0</min_angle>
-              <max_angle>0</max_angle>
-            </horizontal>
-          </scan>
-          <range>
-            <min>0.01</min>
-            <max>0.04</max>
-            <resolution>0.1</resolution>
-          </range>
-        </ray>
-      </sensor>
-    </gazebo>
-  </xacro:macro>
 </robot>

File: create_description/urdf/rplidar.urdf.xacro (robot description, xacro)
@@ -4,62 +4,54 @@
 	<link name="laser">
 		<collision>
-			<origin xyz="0 0 0" rpy="0 0 0"/>
+			<origin xyz="0 0 0" rpy="0 0 0" />
 			<geometry>
-				<box size="0.1 0.1 0.1"/>
+				<box size="0.1 0.1 0.1" />
 			</geometry>
 		</collision>
 		<vision>
-			<origin xyz="0 0 0.1" rpy="1.5707 0 0"/>
+			<origin xyz="0 0 0.1" rpy="1.5707 0 0" />
 			<geometry>
-				<box size="0.1 0.1 0.1"/>
+				<box size="0.1 0.1 0.1" />
 				<meshfile name="package://create_description/meshes/rplidar.dae" scale="0.001 0.001 0.001" />
 			</geometry>
 		</vision>
 		<inertial>
-			<mass value="1e-5"/>
-			<origin xyz="0 0 0" rpy="0 0 0"/>
-			<inertia ixx="1e-6" ixy="0" ixz="0" iyy="1e-6" iyz="0" izz="1e-6"/>
+			<mass value="1e-5" />
+			<origin xyz="0 0 0" rpy="0 0 0" />
+			<inertia ixx="1e-6" ixy="0" ixz="0" iyy="1e-6" iyz="0" izz="1e-6" />
 		</inertial>
 	</link>
 	<joint name="rplidar_joint" type="fixed">
-		<axis xyz="0 1 0"/>
-		<origin xyz="0 0 0.1" rpy="0 0 0 "/>
-		<parent link="base_link"/>
-		<child link="laser"/>
+		<axis xyz="0 1 0" />
+		<origin xyz="0 0 0.1" rpy="0 0 0 " />
+		<parent link="base_link" />
+		<child link="laser" />
 	</joint>
-<gazebo reference="laser">
-	<sensor type="ray" name="head_rplidar_sensor">
-		<pose>0 0 0 0 0 0</pose>
-		<visualize>true</visualize>
-		<update_rate>10</update_rate>
-		<ray>
-			<scan>
-				<horizontal>
-					<samples>360</samples>
-					<min_angle>-3.14159</min_angle>
-					<max_angle>3.14159</max_angle>
-				</horizontal>
-			</scan>
-			<range>
-				<min>0.15</min>
-				<max>4.0</max>
-				<resolution>0.01</resolution>
-			</range>
-			<noise>
-				<type>gaussian</type>
-				<mean>0.0</mean>
-				<stddev>0.01</stddev>
-			</noise>
-		</ray>
-		<plugin name="gazebo_ros_rplidar_controller" filename="libgazebo_ros_ray_sensor.so">
-			<topic_name>/scan</topic_name>
-            <output_type>sensor_msgs/LaserScan</output_type>
-			<frame_name>laser</frame_name>
-            <ros>
-                <namespace></namespace>
-                <remapping>~/out:=scan</remapping>
-            </ros>
-		</plugin>
-	</sensor>
-</gazebo>
+	<gazebo reference="laser">
+		<sensor name='gpu_lidar' type='gpu_lidar'>
+			<ignition_frame_id>laser</ignition_frame_id>
+			<topic>scan</topic>
+			<update_rate>10</update_rate>
+			<lidar>
+				<scan>
+					<horizontal>
+						<samples>360</samples>
+						<min_angle>-3.14159</min_angle>
+						<max_angle>3.14159</max_angle>
+					</horizontal>
+				</scan>
+				<range>
+					<min>0.15</min>
+					<max>4.0</max>
+					<resolution>0.01</resolution>
+				</range>
+				<noise>
+					<type>gaussian</type>
+					<mean>0.0</mean>
+					<stddev>0.01</stddev>
+				</noise>
+			</lidar>
+			<visualize>true</visualize>
+		</sensor>
+	</gazebo>
 </robot>
